File: horno.kicad_sch (KiCad schematic)
At the start: 9 parts, among them U2 STM32F103C8Tx

Commit message: com
Parts:
- removed C5 (x4): 100n, Capacitor_THT:CP_Radial_D8.0mm_P3.80mm, symbol Device:C
- removed Power1: Conn_01x05_Pin, Connector_PinHeader_2.54mm:PinHeader_1x05_P2.54mm_Vertical, symbol Connector:Conn_01x05_Pin
- removed usart1: Conn_01x04_Pin, Connector_PinHeader_2.54mm:PinHeader_1x04_P2.54mm_Vertical, symbol Connector:Conn_01x04_Pin
- added C8 (x4): 100n, Capacitor_SMD:C_1210_3225Metric, symbol Device:C
- added PWR1: Conn_01x16_Pin, Connector_PinHeader_2.54mm:PinHeader_1x16_P2.54mm_Horizontal, symbol Connector:Conn_01x16_Pin
- added Q1, Q2: BC848, Package_TO_SOT_SMD:SOT-23, symbol Transistor_BJT:BC848
- added R1, R2: 4.7k, Resistor_SMD:R_0805_2012Metric, symbol Device:R
- added USART1: Conn_01x05_Pin, Connector_PinHeader_2.54mm:PinHeader_1x05_P2.54mm_Vertical, symbol Connector:Conn_01x05_Pin
- renumbered U2 to U1
Connections:
- net 0: now also Display1.1 (Pin_1), Encoder_Switch1.2 (Pin_2), C8.1, C8.2, C8.2, C8.2, PWR1.4 (Pin_4), Q1.2 (E), Q2.2 (E), USART1.1 (Pin_1); no longer Display1.2 (Pin_2), Encoder_Switch1.1 (Pin_1)
- net 3.3V: now also Display1.2 (Pin_2), Encoder_Switch1.1 (Pin_1), C8.1, C8.1, C8.2, USART1.2 (Pin_2); no longer Display1.1 (Pin_1), Display1.8 (Pin_8), Encoder_Switch1.2 (Pin_2)
- net 5V: now also C8.1, PWR1.3 (Pin_3)
- net IN_OK: now reaches Encoder_Switch1.3 (Pin_3), U1.45 (PB8)
- net IN_CH2: now reaches Encoder_Switch1.4 (Pin_4), U1.43 (PB7)
- net IN_CH1: now reaches Encoder_Switch1.5 (Pin_5), U1.42 (PB6)
- net USART_RX: now reaches U1.31 (PA10)
- net USART_RX: now also USART1.3 (Pin_3)
- net USART_TX: now reaches U1.30 (PA9)
- net USART_TX: now also USART1.4 (Pin_4)
- net USART_CLK: now reaches U1.29 (PA8)
- net USART_CLK: now also USART1.5 (Pin_5)
- net at U1.25 (PB12): now also R2.1
- net at U1.26 (PB13): now also R1.1
- net PWR_ZC: now reaches U1.27 (PB14)
- net PWR_ZC: now also PWR1.12 (Pin_12)
- net LCD_CS: now reaches Display1.3 (Pin_3), U1.22 (PB11)
- net LCD_RST: now reaches Display1.4 (Pin_4), U1.21 (PB10)
- net LCD_DC: now reaches Display1.5 (Pin_5), U1.19 (PB1)
- net LCD_MOSI: now reaches Display1.6 (Pin_6), U1.17 (PA7)
- net LCD_CLK: now reaches Display1.7 (Pin_7), U1.15 (PA5)
- net LCD_MISO: now reaches Display1.9 (Pin_9), U1.16 (PA6)
- net LCD_LED: now reaches U1.18 (PB0)
- net LCD_LED: now also Display1.8 (Pin_8)
- new net: Q1.1 (B), R1.2
- new net: Q2.1 (B), R2.2
- new net PWR_CH1: PWR1.10 (Pin_10), Q2.3 (C)
- new net PWR_CH2: PWR1.11 (Pin_11), Q1.3 (C)
Other:
- moved on the sheet: Display1, Encoder_Switch1
